File: hardware/vu_leds/vu_leds/vu_leds.kicad_pcb (KiCad board)
At the start: 2 copper layers, 80 x 42.5 mm, 19 parts, among them J1 Conn_01x10_Male

Commit message: pdf of pcb layout
Other:
- board outline removed

Commit message: made pcb smaller
Parts:
- moved R8 11.1 mm to (123.4, 109.5), turned to 0 degrees
- moved R3 10.3 mm to (108.0, 109.5), turned to 180 degrees
- moved R9 5.71 mm to (135.4, 103.1)
- moved R1 5.09 mm to (89.7, 104.9), turned to 0 degrees
- moved R2 4.73 mm to (89.7, 109.5), turned to 0 degrees
- moved R7 3.25 mm to (123.4, 104.9), turned to 0 degrees
- moved R6 2.72 mm to (117.6, 103.4)
- moved R4 2.33 mm to (108.0, 104.9), turned to 180 degrees
- moved R5 1.82 mm to (113.0, 103.4)
Routing:
- net Net-(J1-Pad10): track 103.9 -> 90.5 mm
- net Net-(D3-Pad1): track 7.21 -> 15.5 mm
- net Net-(D9-Pad1): track 14.1 -> 8.21 mm
- net Net-(D2-Pad1): track 8.00 -> 13.1 mm
- net Net-(D1-Pad1): track 10.4 -> 6.43 mm
- net Net-(D6-Pad1): track 9.17 -> 5.77 mm
- net Net-(D7-Pad1): track 10.5 -> 7.61 mm
- net Net-(D8-Pad1): track 11.1 -> 12.9 mm
- net Net-(D5-Pad1): track 7.60 -> 5.98 mm
- net Net-(D4-Pad1): track 6.80 -> 7.51 mm
