File: hardware/mic-ampv1/mic-ampv1.kicad_sch (KiCad schematic)
At the start: 16 parts, among them J1 XLR3_Switched, U1 NE5532

Commit message: Updated mic preamp. Increased gain. larger PCB
Parts:
- C1, C2: footprint Capacitor_THT:C_Disc_D3.0mm_W2.0mm_P2.50mm -> Capacitor_THT:C_Rect_L7.0mm_W2.0mm_P5.00mm
Connections:
- net at R5.1, R7.2, RV1.1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: now also RV1.2
- net at R6.1, RV1.3: no longer RV1.2
Changed lines of the file:
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@@
-	)
-	(junction
-		(at 174.752 95.758)
-		(diameter 0)
-		(color 0 0 0 0)
 	)
 	(junction
@@
 	(wire
 		(pts
+			(xy 184.15 100.33) (xy 184.15 96.52)
+		)
+		(stroke
+			(width 0)
+			(type default)
+		)
+	)
+	(wire
+		(pts
 			(xy 173.228 56.388) (xy 173.228 62.738)
 		)
@@
 	(wire
 		(pts
-			(xy 174.752 99.568) (xy 174.752 95.758)
-		)
-		(stroke
-			(width 0)
-			(type default)
-		)
-	)
-	(wire
-		(pts
 			(xy 201.93 82.042) (xy 201.93 81.788)
 		)
@@
 	(wire
 		(pts
+			(xy 184.15 100.33) (xy 178.562 100.33)
+		)
+		(stroke
+			(width 0)
+			(type default)
+		)
+	)
+	(wire
+		(pts
 			(xy 117.856 106.172) (xy 125.476 106.172)
 		)
@@
 	(wire
 		(pts
-			(xy 178.562 99.568) (xy 174.752 99.568)
-		)
-		(stroke
-			(width 0)
-			(type default)
-		)
-	)
-	(wire
-		(pts
 			(xy 63.754 83.312) (xy 85.344 83.312)
 		)
@@
 	(wire
 		(pts
+			(xy 184.15 96.52) (xy 186.69 96.52)
+		)
+		(stroke
+			(width 0)
+			(type default)
+		)
+	)
+	(wire
+		(pts
 			(xy 199.644 45.212) (xy 187.706 45.212)
 		)
@@
 	(wire
 		(pts
+			(xy 178.562 100.33) (xy 178.562 99.568)
+		)
+		(stroke
+			(width 0)
+			(type default)
+		)
+	)
+	(wire
+		(pts
 			(xy 85.344 83.312) (xy 85.344 90.678)
 		)
@@
 		(pts
 			(xy 125.476 90.678) (xy 125.476 97.282)
+		)
+		(stroke
+			(width 0)
+			(type default)
+		)
+	)
+	(wire
+		(pts
+			(xy 186.69 95.758) (xy 186.69 96.52)
 		)
 		(stroke
@@
 			)
 		)
-		(property "Footprint" "Capacitor_THT:C_Disc_D3.0mm_W2.0mm_P2.50mm"
+		(property "Footprint" "Capacitor_THT:C_Rect_L7.0mm_W2.0mm_P5.00mm"
 			(at 87.63 91.6432 0)
 			(effects
@@
 			)
 		)
-		(property "Footprint" "Capacitor_THT:C_Disc_D3.0mm_W2.0mm_P2.50mm"
+		(property "Footprint" "Capacitor_THT:C_Rect_L7.0mm_W2.0mm_P5.00mm"
 			(at 87.63 79.9592 0)
 			(effects
