File: hardware/mixer/4ch_mixer.kicad_sch (KiCad schematic)
At the start: 34 parts, among them J1-Mic1 Conn_01x02_Pin, J1-pwr1 PWR, J2-Mic2 Conn_01x02_Pin, J3-Guitar1 Conn_01x02_Pin, J4-Line-In1 Conn_01x02_Pin, J5-Out1 Conn_01x02_Pin, J6-phones1 Phones, U1 NE5532, U2 NE5532, U3 NE5532

Commit message: changing for 5k8 pots and increased gain
Parts:
- removed C5, C6: 0.1uF, Capacitor_THT:C_Rect_L11.0mm_W2.8mm_P10.00mm_MKT, symbol Device:C
- removed J6-phones1: Phones, Connector:FanPinHeader_1x03_P2.54mm_Vertical, symbol Connector:Conn_01x03_Pin
- removed R10, R11: 47R, Resistor_THT:R_Axial_DIN0204_L3.6mm_D1.6mm_P5.08mm_Horizontal, symbol Device:R
- removed R12, R13: 100k, Resistor_THT:R_Axial_DIN0204_L3.6mm_D1.6mm_P5.08mm_Horizontal, symbol Device:R
- removed R8, R9: 1K, Resistor_THT:R_Axial_DIN0204_L3.6mm_D1.6mm_P5.08mm_Horizontal, symbol Device:R
- removed RV5: 10K, Connector_PinHeader_2.54mm:PinHeader_1x03_P2.54mm_Vertical, symbol Device:R_Potentiometer
- removed unit 1 of U3
- removed unit 2 of U3
- J1-Mic1, J2-Mic2, J3-Guitar1, J4-Line-In1, J5-Out1: footprint Connector_PinHeader_2.54mm:PinHeader_1x02_P2.54mm_Vertical -> Connector_JST:JST_EH_B2B-EH-A_1x02_P2.50mm_Vertical
- J1-pwr1: footprint Connector:FanPinHeader_1x03_P2.54mm_Vertical -> Connector_JST:JST_EH_B3B-EH-A_1x03_P2.50mm_Vertical
- R1, R2, R3: value 100k -> 5K6
- R4, R5: value 100k -> 5k6
- R6: value 100k -> 10k
- RV1, RV2, RV3, RV4: value 100K -> 5K8; footprint Connector_PinHeader_2.54mm:PinHeader_1x03_P2.54mm_Vertical -> Connector_JST:JST_EH_B3B-EH-A_1x03_P2.50mm_Vertical
